File: PTP_David_Hanzir_Projekt1/PTP_David_Hanzir_Projekt1.kicad_sch (KiCad schematic)
At the start: 3 parts, among them U1 NUCLEO64-F411RE

Commit message: LV2
Parts:
- removed U1: NUCLEO64-F411RE, Module:ST_Morpho_Connector_144_STLink, symbol MCU_Module:NUCLEO64-F411RE
- added C3: 22u, symbol Device:C_Polarized
- added C4, C8: 100u, symbol Device:C
- added C6: 220u, symbol Device:C_Polarized
- added C7: 10u, symbol Device:C
- added D1, D3, D4, D5: LED, symbol Device:LED
- added D2: 11DQ06, symbol Device:D_Schottky_Filled
- added J1: Screw_Terminal_01x02, symbol Connector:Screw_Terminal_01x02
- added L1: 330u, symbol Device:L
- added R3, R4, R5, R6, R7, R8: 47k, symbol Device:R_Small
- added SW1: ~, symbol Switch:SW_Push
- added SW2: ~, symbol Switch:SW_SPDT
- added U1: NE555P, Package_DIP:DIP-8_W7.62mm, symbol Timer:NE555P
- added U2: LM2574N-5, Package_DIP:DIP-8_W7.62mm, symbol Regulator_Switching:LM2574N-5
- R1, R2: value R_Small -> 2k
Connections:
- net GND: now also C3.2, C4.1, C6.2, C7.2, C8.2, D2.2 (A), J1.1 (Pin_1), R5.2, R6.2, R7.2, R8.2, SW1.1, U2.2 (SGND), U2.3 (~{ON}/OFF), U2.4 (PGND); no longer R2.1
- net +3.3V: no longer names the net of R1.2
- net +3.3V: now also R2.2, C4.2, SW2.3 (C)
- net u_Izl renamed +5V
- net +5V: now also C6.1, C8.1, L1.2, R3.1, U1.8 (VCC), U2.1 (FB); no longer R2.2
- new net: C7.1, R4.2, U1.2 (TR), U1.6 (THR)
- new net: R3.2, R4.1, U1.7 (DIS)
- new net: D2.1 (K), L1.1, U2.7 (OUT)
- new net: R2.1, SW1.2
- new net: D4.1 (K), R7.1
- new net: D3.1 (K), R6.1
- new net: D1.1 (K), R5.1
- new net: D5.1 (K), R8.1
- new net 555: SW2.2 (A), U1.3 (Q)
- new net Clock: SW2.1 (B)
- new net Q0: D1.2 (A)
- new net Q1: D3.2 (A)
- new net Q2: D4.2 (A)
- new net Q3: D5.2 (A)
- new net VD: C3.1, J1.2 (Pin_2), U2.5 (VIN)
- no-connect marks 2 -> 0

Commit message: LV3
Parts:
- removed C4: 100u, symbol Device:C
- removed R1, R2: 2k, symbol Device:R_Small
- removed SW1: ~, symbol Switch:SW_Push
- removed SW2: ~, symbol Switch:SW_SPDT
- added C1: 100u, symbol Device:C
- added R7: 10, symbol Device:R_Small
- added R9: 2k, symbol Device:R_Small
- added SW3: SW3, symbol Switch:SW_Push
- added SW4: ~, symbol Switch:SW_SPDT
- added U3: ~, symbol SN74LVC1G11:SN74LVC1G11
- J1: value Screw_Terminal_01x02 -> ~
- R1: renamed from R5; value 47k -> 4k7
- R2: renamed from R6; value 47k -> 4k7
- R3: renamed from R7; value 47k -> 4k7
- R4: renamed from R8; value 47k -> 4k7
- renumbered C3 to C1, C6 to C2, D3 to D2, D4 to D3, D2 to D4, U2 to U1
Connections:
- net +5V: now also R7.1, U3.5 (VCC)
- net 555: now also SW4.2 (A)
- net Clock: now also R7.2, SW4.1 (B), U3.6
- net GND: now also C1.1, SW3.1, U3.2 (GND)
- net Q1: now also U3.1
- net Q2: now also U3.3
- new net: R9.1, SW3.2
- new net: C1.2, R9.2, SW4.3 (C)
- new net Reset: U3.4 (Y)

Commit message: LV4
Parts:
- added H1, H2, H3, H4: MountingHole, symbol Mechanical:MountingHole
- added R10, R11, R12, R15, R9: 10k, symbol Device:R_Small
- added R14, R16, R17, R18, R5, R6, R8: 2k, symbol Device:R_Small
- added U2, U3: 4027, Package_DIP:DIP-16_W7.62mm_Socket_LongPads, symbol 4xxx:4027
- added U4: 74LS47, Package_DIP:DIP-16_W7.62mm_Socket_LongPads, symbol 74xx:74LS47
- added U5: HDSP-7401, Display_7Segment:HDSP-7401, symbol Display_Character:HDSP-7401
- U1: footprint Package_DIP:DIP-8_W7.62mm -> Package_DIP:DIP-8_W7.62mm_Socket_LongPads; Manufacturer (none) -> ONSEMI; Manufacturer Part Number  (none) -> LM2574N-5G
- U6: renamed from U3; value ~ -> 74lLVC1G11
- U7: renamed from U1; Manufacturer (none) -> TEXAS INSTRUMENTS; Manufacturer Part Number  (none) -> NE555P
- renumbered C7 to C6, C8 to C7, C1 to C8, C1 to C9, R3 to R19, R4 to R20
Connections:
- net +5V: now also U7.4 (R), R10.1, R11.1, R12.1, R15.1, R9.1, U2.16 (VDD), U3.16 (VDD), U4.16 (VCC), U5.1 (CA), U5.6 (CA)
- net Clock: now also U6.3, U2.3 (C); no longer U6.6
- net GND: now also U7.1 (GND), U2.7 (S), U2.8 (VSS), U2.9 (S), U3.7 (S), U3.8 (VSS), U3.9 (S), U4.8 (GND)
- net Q0: now also U2.1 (Q), U2.13 (C), U4.7 (A)
- net Q1: now also U6.6, U2.15 (Q), U3.3 (C), U4.1 (B); no longer U6.1
- net Q2: now also U3.1 (Q), U3.13 (C), U4.2 (C); no longer U6.3
- net Q3: now also U6.1, U3.15 (Q), U4.6 (D)
- net Reset: now also U2.12 (R), U2.4 (R), U3.12 (R), U3.4 (R)
- new net: R5.1, U4.13 (a)
- new net: R5.2, U5.10 (A)
- new net: R18.1, U4.14 (g)
- new net: R18.2, U5.3 (G)
- new net: R9.2, U2.5 (K), U2.6 (J)
- new net: R14.1, U4.10 (d)
- new net: R14.2, U5.5 (D)
- new net: R6.1, U4.12 (b)
- new net: R6.2, U5.9 (B)
- new net: R16.1, U4.9 (e)
- new net: R16.2, U5.4 (E)
- new net: R11.2, U3.5 (K), U3.6 (J)
- new net: R10.2, U2.10 (J), U2.11 (K)
- new net: R12.2, U3.10 (J), U3.11 (K)
- new net: R8.1, U4.11 (c)
- new net: R17.1, U4.15 (f)
- new net: R15.2, U4.3 (LT), U4.4 (BI), U4.5 (RBI)
- new net: R17.2, U5.2 (F)
- new net: R8.2, U5.8 (C)
- no-connect marks 0 -> 6
Other:
- note added: "555 timer"
- note added: "JK bistabili"
- note added: "LED diode"
- note added: "Montažne rupe"
- note added: "Napajanje"
- note added: "Napajanje bistabila"
- note added: "Reset brojača"
- note added: "Tipkalo i ulaz radnog takta"
- company: (none) -> Tehničko veleučilište u Zagrebu
- title: (none) -> BCD Brojač
- moved on the sheet: U6

Commit message: LV5
Parts:
- C1: renamed from C9; footprint (none) -> Capacitor_THT:CP_Radial_D5.0mm_P2.00mm
- C2: footprint (none) -> Capacitor_THT:CP_Radial_D5.0mm_P2.00mm
- C3: renamed from C8; footprint (none) -> Capacitor_SMD:C_1206_3216Metric_Pad1.33x1.80mm_HandSolder
- C4: renamed from C7; footprint (none) -> Capacitor_SMD:C_1206_3216Metric_Pad1.33x1.80mm_HandSolder
- C5: renamed from C6; footprint (none) -> Capacitor_SMD:C_1206_3216Metric_Pad1.33x1.80mm_HandSolder
- D1, D2, D3, D5: footprint (none) -> LED_THT:LED_D5.0mm
- D4: footprint (none) -> Diode_THT:D_DO-41_SOD81_P12.70mm_Horizontal
- H1, H2, H3, H4: footprint (none) -> MountingHole:MountingHole_5.5mm
- J1: footprint (none) -> TerminalBlock_MetzConnect:TerminalBlock_MetzConnect_Type011_RT05502HBLC_1x02_P5.00mm_Horizontal
- L1: footprint (none) -> Inductor_THT:L_Radial_D7.2mm_P3.00mm_Murata_1700
- R1, R2, R3, R4: footprint (none) -> Resistor_THT:R_Axial_DIN0207_L6.3mm_D2.5mm_P10.16mm_Horizontal
- R10, R11, R12, R14, R15, R16, R17, R18, R19, R20, R5, R6, R7, R8, R9: footprint (none) -> Resistor_SMD:R_1206_3216Metric_Pad1.30x1.75mm_HandSolder
- R13: renamed from R9; footprint (none) -> Resistor_SMD:R_1206_3216Metric_Pad1.30x1.75mm_HandSolder
- SW1: renamed from SW3; value SW3 -> SW1; footprint (none) -> Button_Switch_THT:SW_PUSH_6mm_H4.3mm
- SW2: renamed from SW4; footprint (none) -> Button_Switch_THT:SW_Slide_SPDT_Straight_CK_OS102011MS2Q
- U6: footprint (none) -> Package_TO_SOT_SMD:SOT-23-6; Manufacturer (none) -> TEXAS INSTRUMENTS; Manufacturer Part Number  (none) -> SN74LVC1G11DBVR SN74LVC1G11DBVR
Changed lines of the file:
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@@
 			)
 		)
-		(property "Footprint" ""
+		(property "Footprint" "Resistor_SMD:R_1206_3216Metric_Pad1.30x1.75mm_HandSolder"
 			(at 193.04 92.71 0)
 			(effects
@@
 		(dnp no)
 		(fields_autoplaced yes)
-		(property "Reference" "R9"
+		(property "Reference" "R13"
 			(at 245.11 38.1 90)
 			(effects
@@
 			)
 		)
-		(property "Footprint" ""
+		(property "Footprint" "Resistor_SMD:R_1206_3216Metric_Pad1.30x1.75mm_HandSolder"
 			(at 245.11 43.18 0)
 			(effects
@@
 			(project "PTP_David_Hanzir_Projekt1"
 				(path "/a4d2f06c-c791-4317-8d5f-152a30bd9a0f"
-					(reference "R9")
+					(reference "R13")
 					(unit 1)
 				)
@@
 			)
 		)
-		(property "Footprint" ""
+		(property "Footprint" "Resistor_SMD:R_1206_3216Metric_Pad1.30x1.75mm_HandSolder"
 			(at 193.04 123.19 0)
 			(effects
@@
 			)
 		)
-		(property "Footprint" ""
+		(property "Footprint" "Inductor_THT:L_Radial_D7.2mm_P3.00mm_Murata_1700"
 			(at 193.04 41.91 0)
 			(effects
@@
 		(dnp no)
 		(fields_autoplaced yes)
-		(property "Reference" "C9"
+		(property "Reference" "C1"
 			(at 132.08 44.8309 0)
 			(effects
@@
 			)
 		)
-		(property "Footprint" ""
+		(property "Footprint" "Capacitor_THT:CP_Radial_D5.0mm_P2.00mm"
 			(at 129.2352 50.8 0)
 			(effects
@@
 			(project ""
 				(path "/a4d2f06c-c791-4317-8d5f-152a30bd9a0f"
-					(reference "C9")
+					(reference "C1")
 					(unit 1)
 				)
@@
 			)
 		)
-		(property "Footprint" ""
+		(property "Footprint" "LED_THT:LED_D5.0mm"
 			(at 39.37 119.38 0)
 			(effects
@@
 			)
 		)
-		(property "Footprint" ""
+		(property "Footprint" "MountingHole:MountingHole_5.5mm"
 			(at 147.32 171.45 0)
 			(effects
@@
 			)
 		)
-		(property "Footprint" ""
+		(property "Footprint" "Resistor_SMD:R_1206_3216Metric_Pad1.30x1.75mm_HandSolder"
 			(at 27.94 170.18 0)
 			(effects
@@
 			)
 		)
-		(property "Footprint" ""
+		(property "Footprint" "MountingHole:MountingHole_5.5mm"
 			(at 147.32 163.83 0)
 			(effects
@@
 		(dnp no)
 		(fields_autoplaced yes)
-		(property "Reference" "C6"
+		(property "Reference" "C5"
 			(at 27.94 71.1199 0)
 			(effects
@@
 			)
 		)
-		(property "Footprint" ""
+		(property "Footprint" "Capacitor_SMD:C_1206_3216Metric_Pad1.33x1.80mm_HandSolder"
 			(at 25.0952 76.2 0)
 			(effects
@@
 			(project "PTP_David_Hanzir_Projekt1"
 				(path "/a4d2f06c-c791-4317-8d5f-152a30bd9a0f"
-					(reference "C6")
+					(reference "C5")
 					(unit 1)
 				)
@@
 			)
 		)
-		(property "Footprint" ""
+		(property "Footprint" "Resistor_THT:R_Axial_DIN0207_L6.3mm_D2.5mm_P10.16mm_Horizontal"
 			(at 53.34 111.76 0)
 			(effects
@@
 		(dnp no)
 		(fields_autoplaced yes)
-		(property "Reference" "C8"
+		(property "Reference" "C3"
 			(at 238.76 24.13 90)
 			(effects
@@
 			)
 		)
-		(property "Footprint" ""
+		(property "Footprint" "Capacitor_SMD:C_1206_3216Metric_Pad1.33x1.80mm_HandSolder"
 			(at 242.57 30.7848 0)
 			(effects
@@
 			(project "PTP_David_Hanzir_Projekt1"
 				(path "/a4d2f06c-c791-4317-8d5f-152a30bd9a0f"
-					(reference "C8")
+					(reference "C3")
 					(unit 1)
 				)
@@
 			)
 		)
-		(property "Footprint" ""
+		(property "Footprint" "Resistor_SMD:R_1206_3216Metric_Pad1.30x1.75mm_HandSolder"
 			(at 193.04 107.95 0)
 			(effects
@@
 			)
 		)
-		(property "Footprint" ""
+		(property "Footprint" "Resistor_THT:R_Axial_DIN0207_L6.3mm_D2.5mm_P10.16mm_Horizontal"
 			(at 53.34 104.14 0)
 			(effects
@@
 			)
 		)
-		(property "Footprint" ""
+		(property "Footprint" "Resistor_SMD:R_1206_3216Metric_Pad1.30x1.75mm_HandSolder"
 			(at 193.04 97.79 0)
 			(effects
@@
 		(dnp no)
 		(fields_autoplaced yes)
-		(property "Reference" "SW4"
+		(property "Reference" "SW2"
 			(at 266.7 36.83 0)
 			(effects
@@
 			)
 		)
-		(property "Footprint" ""
+		(property "Footprint" "Button_Switch_THT:SW_Slide_SPDT_Straight_CK_OS102011MS2Q"
 			(at 266.7 45.72 0)
 			(effects
@@
 			(project "PTP_David_Hanzir_Projekt1"
 				(path "/a4d2f06c-c791-4317-8d5f-152a30bd9a0f"
-					(reference "SW4")
+					(reference "SW2")
 					(unit 1)
 				)
@@
 			)
 		)
-		(property "Footprint" ""
+		(property "Footprint" "MountingHole:MountingHole_5.5mm"
 			(at 147.32 187.96 0)
 			(effects
@@
 		(dnp no)
 		(fields_autoplaced yes)
-		(property "Reference" "C7"
+		(property "Reference" "C4"
 			(at 40.64 43.1799 0)
 			(effects
@@
 			)
 		)
-		(property "Footprint" ""
+		(property "Footprint" "Capacitor_SMD:C_1206_3216Metric_Pad1.33x1.80mm_HandSolder"
 			(at 37.7952 48.26 0)
 			(effects
@@
 			(project ""
 				(path "/a4d2f06c-c791-4317-8d5f-152a30bd9a0f"
-					(reference "C7")
+					(reference "C4")
 					(unit 1)
 				)
@@
 			)
 		)
-		(property "Footprint" ""
+		(property "Footprint" "TerminalBlock_MetzConnect:TerminalBlock_MetzConnect_Type011_RT05502HBLC_1x02_P5.00mm_Horizontal"
 			(at 105.41 36.83 0)
 			(effects
@@
 			)
 		)
-		(property "Footprint" ""
+		(property "Footprint" "Resistor_SMD:R_1206_3216Metric_Pad1.30x1.75mm_HandSolder"
 			(at 193.04 113.03 0)
 			(effects
@@
 			)
 		)
-		(property "Footprint" ""
+		(property "Footprint" "Diode_THT:D_DO-41_SOD81_P12.70mm_Horizontal"
 			(at 184.15 54.61 0)
 			(effects
@@
 			)
 		)
-		(property "Footprint" ""
+		(property "Footprint" "LED_THT:LED_D5.0mm"
 			(at 39.37 111.76 0)
 			(effects
@@
 			)
 		)
-		(property "Footprint" ""
+		(property "Footprint" "MountingHole:MountingHole_5.5mm"
 			(at 147.32 180.34 0)
 			(effects
@@
 			)
 		)
-		(property "Footprint" ""
+		(property "Footprint" "LED_THT:LED_D5.0mm"
 			(at 39.37 104.14 0)
 			(effects
@@
 			)
 		)
-		(property "Footprint" ""
+		(property "Footprint" "Resistor_SMD:R_1206_3216Metric_Pad1.30x1.75mm_HandSolder"
 			(at 104.14 171.45 0)
 			(effects
@@
 			)
 		)
-		(property "Footprint" ""
+		(property "Footprint" "Resistor_SMD:R_1206_3216Metric_Pad1.30x1.75mm_HandSolder"
 			(at 77.47 171.45 0)
 			(effects
@@
 			)
 		)
-		(property "Footprint" ""
+		(property "Footprint" "Resistor_SMD:R_1206_3216Metric_Pad1.30x1.75mm_HandSolder"
 			(at 24.13 59.69 0)
 			(effects
@@
 			)
 		)
-		(property "Footprint" ""
+		(property "Footprint" "Resistor_SMD:R_1206_3216Metric_Pad1.30x1.75mm_HandSolder"
 			(at 273.05 36.83 0)
 			(effects
@@
 			)
 		)
-		(property "Footprint" ""
+		(property "Footprint" "Resistor_SMD:R_1206_3216Metric_Pad1.30x1.75mm_HandSolder"
 			(at 24.13 45.72 0)
 			(effects
@@
 			)
 		)
-		(property "Footprint" ""
+		(property "Footprint" "Resistor_THT:R_Axial_DIN0207_L6.3mm_D2.5mm_P10.16mm_Horizontal"
 			(at 53.34 119.38 0)
 			(effects
@@
 			)
 		)
-		(property "Footprint" ""
+		(property "Footprint" "LED_THT:LED_D5.0mm"
 			(at 39.37 127 0)
 			(effects
@@
 			)
 		)
-		(property "Footprint" ""
+		(property "Footprint" "Resistor_SMD:R_1206_3216Metric_Pad1.30x1.75mm_HandSolder"
 			(at 138.43 113.03 0)
 			(effects
@@
 			)
 		)
-		(property "Footprint" ""
+		(property "Footprint" "Resistor_SMD:R_1206_3216Metric_Pad1.30x1.75mm_HandSolder"
 			(at 193.04 102.87 0)
 			(effects
@@
 			)
 		)
-		(property "Footprint" ""
+		(property "Footprint" "Resistor_THT:R_Axial_DIN0207_L6.3mm_D2.5mm_P10.16mm_Horizontal"
 			(at 53.34 127 0)
 			(effects
@@
 			)
 		)
-		(property "Footprint" ""
+		(property "Footprint" "Capacitor_THT:CP_Radial_D5.0mm_P2.00mm"
 			(at 210.5152 55.88 0)
 			(effects
@@
 			)
 		)
-		(property "Footprint" ""
+		(property "Footprint" "Resistor_SMD:R_1206_3216Metric_Pad1.30x1.75mm_HandSolder"
 			(at 53.34 171.45 0)
 			(effects
@@
 		(dnp no)
 		(fields_autoplaced yes)
-		(property "Reference" "SW3"
+		(property "Reference" "SW1"
 			(at 234.95 35.56 0)
 			(effects
@@
 			)
 		)
-		(property "Value" "SW3"
+		(property "Value" "SW1"
 			(at 234.95 38.1 0)
 			(effects
@@
 			)
 		)
-		(property "Footprint" ""
+		(property "Footprint" "Button_Switch_THT:SW_PUSH_6mm_H4.3mm"
 			(at 234.95 38.1 0)
 			(effects
@@
 			(project "PTP_David_Hanzir_Projekt1"
 				(path "/a4d2f06c-c791-4317-8d5f-152a30bd9a0f"
-					(reference "SW3")
+					(reference "SW1")
 					(unit 1)
 				)
@@
 			)
 		)
-		(property "Footprint" ""
+		(property "Footprint" "Package_TO_SOT_SMD:SOT-23-6"
 			(at 107.95 121.92 0)
 			(effects
@@
 			)
 		)
+		(property "Manufacturer" "TEXAS INSTRUMENTS "
+			(at 107.95 121.92 0)
+			(effects
+				(font
+					(size 1.27 1.27)
+				)
+				(hide yes)
+			)
+		)
+		(property "Manufacturer Part Number " "SN74LVC1G11DBVR SN74LVC1G11DBVR "
+			(at 107.95 121.92 0)
+			(effects
+				(font
+					(size 1.27 1.27)
+				)
+				(hide yes)
+			)
+		)
 		(pin "1"
 		)
@@
 			)
 		)
-		(property "Footprint" ""
+		(property "Footprint" "Resistor_SMD:R_1206_3216Metric_Pad1.30x1.75mm_HandSolder"
 			(at 193.04 118.11 0)
 			(effects
